Commit message: change urdf

File: src/spider_rl_mjlab/assets/phybot_c2/urdf/phybot_c2.urdf (robot description, URDF)
Before this commit: robot phybot_c2, 27 links, 26 joints
Links:
- added link left_hand_spine, mass 1; collision box size=0.12 0.012 0.2573595; visual mesh filename=meshes/left_hand_spine.stl
- added link right_hand_spine, mass 1; collision box size=0.12 0.012 0.2573595; visual mesh filename=meshes/right_hand_spine.STL
- link base_link: geometry collision sphere radius=0.07; visual mesh filename=meshes/base_link.STL
- link left_ankle_pitch: mass 1.55163108561377 -> 1.5516311; geometry collision sphere radius=0.045; visual mesh filename=meshes/left_ankle_pitch.STL
- link left_ankle_roll: mass 0.388009531160459 -> 0.3880095; geometry collision cylinder length=0.15 radius=0.01; collision cylinder length=0.15 radius=0.01
- link left_elbow_pitch: mass 0.851991701787346 -> 0.8519917; geometry collision cylinder length=0.22 radius=0.035; visual mesh filename=meshes/left_elbow_pitch.STL
- link left_hip_pitch: geometry visual mesh filename=meshes/left_hip_pitch.STL
- link left_hip_roll: geometry collision sphere radius=0.05; visual mesh filename=meshes/left_hip_roll.STL
- link left_hip_yaw: mass 1.00442326218312 -> 1.0044233; geometry collision cylinder length=0.18 radius=0.04; visual mesh filename=meshes/left_hip_yaw.STL
- link left_knee: mass 1.35068107452534 -> 1.3506811; geometry collision cylinder length=0.16 radius=0.04; visual mesh filename=meshes/left_knee.STL
- link left_shoulder_pitch: mass 0.827963272040063 -> 0.8279633; geometry visual mesh filename=meshes/left_shoulder_pitch.STL
- link left_shoulder_roll: mass 0.224784045580485 -> 0.224784; geometry collision sphere radius=0.05; visual mesh filename=meshes/left_shoulder_roll.STL
- link left_shoulder_yaw: mass 1.59289091864703 -> 1.5928909; geometry collision cylinder length=0.14 radius=0.03; visual mesh filename=meshes/left_shoulder_yaw.STL
- link neck_pitch: geometry collision sphere radius=0.07; visual mesh filename=meshes/neck_pitch.STL
- link neck_yaw: mass 0.428619902168844 -> 0.4286199; geometry visual mesh filename=meshes/neck_yaw.STL
- link right_ankle_pitch: mass 1.55163108561377 -> 1.5516311; geometry collision sphere radius=0.045; visual mesh filename=meshes/right_ankle_pitch.STL
- link right_ankle_roll: mass 0.397122220931611 -> 0.3971222; geometry collision cylinder length=0.15 radius=0.01; collision cylinder length=0.15 radius=0.01
- link right_elbow_pitch: mass 0.852091777096898 -> 0.8520918; geometry collision cylinder length=0.22 radius=0.035; visual mesh filename=meshes/right_elbow_pitch.STL
- link right_hip_pitch: mass 0.910416842241314 -> 0.9104168; geometry visual mesh filename=meshes/right_hip_pitch.STL
- link right_hip_roll: mass 0.236808848887827 -> 0.2368088; geometry collision sphere radius=0.05; visual mesh filename=meshes/right_hip_roll.STL
- link right_hip_yaw: mass 1.0044272654158 -> 1.0044273; geometry collision cylinder length=0.18 radius=0.04; visual mesh filename=meshes/right_hip_yaw.STL
- link right_knee: mass 1.35067962196111 -> 1.3506796; geometry collision cylinder length=0.16 radius=0.04; visual mesh filename=meshes/right_knee.STL
- link right_shoulder_pitch: mass 0.827963271957507 -> 0.8279633; geometry visual mesh filename=meshes/right_shoulder_pitch.STL
- link right_shoulder_roll: mass 0.224782671869933 -> 0.2247827; geometry collision sphere radius=0.05; visual mesh filename=meshes/right_shoulder_roll.STL
- link right_shoulder_yaw: mass 1.59289091833568 -> 1.5928909; geometry collision cylinder length=0.14 radius=0.03; visual mesh filename=meshes/right_shoulder_yaw.STL
- link torso: mass 11.89499645954187 -> 11.8949965; geometry collision box size=0.14 0.18 0.28; visual mesh filename=meshes/torso.STL
- link waist_yaw: mass 0.209172570853763 -> 0.2091726; geometry visual mesh filename=meshes/waist_yaw.STL
Joints:
- added joint left_hand_spine: type revolute, parent left_elbow_pitch, child left_hand_spine, origin xyz=-0.04 0 0 rpy=0 3.1415927 -1.5707963, axis 0 0 1, limit lower=-1.57 upper=1.57 effort=100 velocity=10
- added joint right_hand_spine: type revolute, parent right_elbow_pitch, child right_hand_spine, origin xyz=-0.04 0 0 rpy=0 3.1415927 -1.5707963, axis 0 0 1, limit lower=-1.57 upper=1.57 effort=100 velocity=10
- joint left_ankle_roll: origin xyz=0.00029206 0 -0.09 rpy=0 0 0 -> xyz=0.0002921 0 -0.09 rpy=0 0 0
- joint left_shoulder_yaw: origin xyz=-0.00052455 0.0085956 -0.048748 rpy=0.17453 0 0 -> xyz=-0.0005246 0.0085956 -0.048748 rpy=0.17453 0 0
- joint neck_pitch: axis 0 1 0 -> (none); limit lower=-0.61 upper=0.61 effort=30 velocity=98.16 -> (none)
- joint neck_yaw: axis 0 0 1 -> (none); limit lower=-2.62 upper=2.62 effort=30 velocity=98.16 -> (none)
- joint right_shoulder_yaw: origin xyz=-0.00052455 -0.0085956 -0.048748 rpy=-0.17453 0 0 -> xyz=-0.0005246 -0.0085956 -0.048748 rpy=-0.17453 0 0
- joint torso: axis 0 0 0 -> (none)

Commit message: climbing milestone

File: src/spider_rl_mjlab/assets/phybot_c2/urdf/phybot_c2.urdf (robot description, URDF)
Before this commit: robot phybot_c2, 29 links, 28 joints
Links:
- added link left_foot_spine, mass 1; collision box size=0.12 0.012 0.1974; visual mesh filename=meshes/left_foot_spine.stl
- added link right_foot_spine, mass 1; collision box size=0.12 0.012 0.1974; visual mesh filename=meshes/right_foot_spine.stl
Joints:
- added joint left_foot_spine: type fixed, parent left_knee, child left_foot_spine, origin xyz=0.05 0 0 rpy=0 0 1.5707963
- added joint right_foot_spine: type fixed, parent right_knee, child right_foot_spine, origin xyz=0.05 0 0 rpy=0 0 1.5707963
- joint left_hand_spine: axis 0 0 1 -> (none); limit lower=-1.57 upper=1.57 effort=100 velocity=10 -> (none); type revolute -> fixed
- joint right_hand_spine: axis 0 0 1 -> (none); limit lower=-1.57 upper=1.57 effort=100 velocity=10 -> (none); type revolute -> fixed
