Commit message: snapshot(microspine): working-tree state of Aug 11 - Sep 22
Captured verbatim before the 2026-09 cleanup so the archive tag preserves
it: the microspine runtime (empirical unit model, wrench/pad geometry,
contact sensor, surfaces), its packaged empirical table, the CAD-derived
PHYBot C2 model (XML/URDF, constants, new microspine meshes and geometry
manifest) and pyproject package data. No edits beyond staging.

Co-Authored-By: Claude Opus 5.5 <noreply@anthropic.com>

File: src/scr_phybot_mjab/assets/phybot_c2/urdf/phybot_c2.urdf (robot description, URDF)
Before this commit: robot phybot_c2, 31 links, 30 joints
Links:
- removed link left_wrist_yaw
- removed link right_wrist_yaw
- added link left_forearm_pad_mount, mass 0.205979717001; collision box size=0.0799999982118 0.0549193359912 0.074999999255; collision cylinder length=0.035 radius=0.0275
- added link right_forearm_pad_mount, mass 0.205979717001; collision box size=0.0799999982118 0.0549193359912 0.074999999255; collision cylinder length=0.035 radius=0.0275
- link left_elbow_pitch: geometry collision cylinder length=0.120 radius=0.021; visual mesh filename=package://DY-CR1-000 小人形机器人AURDF-A/new_meshes/left_forearm_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
- link left_foot_spine: mass 1 -> 0.186895738903; geometry collision box size=0.0279000083712 0.0150000995849 0.025069218463; collision box size=0.0279000083712 0.0150000995849 0.025069218463
- link left_hand_spine: mass 1 -> 0.186895738903; geometry collision box size=0.0279000083712 0.0150000995849 0.025069218463; collision box size=0.0279000083712 0.0150000995849 0.025069218463
- link right_elbow_pitch: geometry collision cylinder length=0.120 radius=0.021; visual mesh filename=package://DY-CR1-000 小人形机器人AURDF-A/new_meshes/right_forearm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
- link right_foot_spine: mass 1 -> 0.186895738903; geometry collision box size=0.0279000083712 0.0150000995849 0.025069218463; collision box size=0.0279000083712 0.0150000995849 0.025069218463
- link right_hand_spine: mass 1 -> 0.186895738903; geometry collision box size=0.0279000083712 0.0150000995849 0.025069218463; collision box size=0.0279000083712 0.0150000995849 0.025069218463
Joints:
- removed joint left_wrist_yaw
- removed joint right_wrist_yaw
- added joint left_forearm_pad_mount: type fixed, parent left_elbow_pitch, child left_forearm_pad_mount, origin xyz=0.01225 0 -0.243500023365 rpy=3.14159265359 0 1.57079632679
- added joint right_forearm_pad_mount: type fixed, parent right_elbow_pitch, child right_forearm_pad_mount, origin xyz=0.01225 0 -0.243500023365 rpy=3.14159265359 0 1.57079632679
- joint left_foot_spine: origin xyz=0.05 0 0 rpy=0 0 1.5707963 -> xyz=0.068 0 -0.15935 rpy=0 0 1.57079632679
- joint left_hand_spine: origin xyz=-0.04 0 0 rpy=0 3.1415927 -1.5707963 -> xyz=0.01225 0 -0.243500023365 rpy=3.14159265359 0 1.57079632679
- joint right_foot_spine: origin xyz=0.05 0 0 rpy=0 0 1.5707963 -> xyz=0.068 0 -0.15935 rpy=0 0 1.57079632679
- joint right_hand_spine: origin xyz=-0.04 0 0 rpy=0 3.1415927 -1.5707963 -> xyz=0.01225 0 -0.243500023365 rpy=3.14159265359 0 1.57079632679

Commit message: [behavior-preserving] assets: drop unused assets, ROS export leftovers and duplicate meshes
- assets/block, assets/slope, assets/forearm_hand: imported by nothing
  (forearm_hand only by the already-broken scripts/debug_contacts.py)
- phybot_c2: CMakeLists.txt, launch/, config/, export.log from the URDF
  exporter, and simple_stl_face.py (hard-coded foreign paths); package.xml
  stays because build_phybot_microspine_assets.py reads its package name
- phybot_c2/meshes/: 27 of 29 files duplicated new_meshes/, which the MJCF
  already uses; the URDF's 23 meshes/ references now point at new_meshes/
  (base_link and torso switch to the decimated copies the MJCF uses)
- unreferenced clips climb_cycle, climb_cycle_moment_safe_fast and
  mini_walk_backward_{0,1} (AMP lists its clips explicitly); tracked .DS_Store

Verified: cfg dumps 42/42 and compiled-model fingerprints 28/28 identical to
the baseline; pytest 433 passed.

Co-Authored-By: Claude Opus 5.5 <noreply@anthropic.com>

File: src/scr_phybot_mjab/assets/phybot_c2/urdf/phybot_c2.urdf (robot description, URDF)
Before this commit: robot phybot_c2, 31 links, 30 joints
Links:
- link base_link: geometry collision sphere radius=0.07; visual mesh filename=new_meshes/base_link.STL
- link left_ankle_pitch: geometry collision sphere radius=0.045; visual mesh filename=new_meshes/left_ankle_pitch.STL
- link left_ankle_roll: geometry collision cylinder length=0.15 radius=0.01; collision cylinder length=0.15 radius=0.01
- link left_hip_pitch: geometry visual mesh filename=new_meshes/left_hip_pitch.STL
- link left_hip_roll: geometry collision sphere radius=0.05; visual mesh filename=new_meshes/left_hip_roll.STL
- link left_hip_yaw: geometry collision cylinder length=0.18 radius=0.04; visual mesh filename=new_meshes/left_hip_yaw.STL
- link left_knee: geometry collision cylinder length=0.16 radius=0.04; visual mesh filename=new_meshes/left_knee.STL
- link left_shoulder_pitch: geometry visual mesh filename=new_meshes/left_shoulder_pitch.STL
- link left_shoulder_roll: geometry collision sphere radius=0.05; visual mesh filename=new_meshes/left_shoulder_roll.STL
- link left_shoulder_yaw: geometry collision cylinder length=0.14 radius=0.03; visual mesh filename=new_meshes/left_shoulder_yaw.STL
- link neck_pitch: geometry collision sphere radius=0.07; visual mesh filename=new_meshes/neck_pitch.STL
- link neck_yaw: geometry visual mesh filename=new_meshes/neck_yaw.STL
- link right_ankle_pitch: geometry collision sphere radius=0.045; visual mesh filename=new_meshes/right_ankle_pitch.STL
- link right_ankle_roll: geometry collision cylinder length=0.15 radius=0.01; collision cylinder length=0.15 radius=0.01
- link right_hip_pitch: geometry visual mesh filename=new_meshes/right_hip_pitch.STL
- link right_hip_roll: geometry collision sphere radius=0.05; visual mesh filename=new_meshes/right_hip_roll.STL
- link right_hip_yaw: geometry collision cylinder length=0.18 radius=0.04; visual mesh filename=new_meshes/right_hip_yaw.STL
- link right_knee: geometry collision cylinder length=0.16 radius=0.04; visual mesh filename=new_meshes/right_knee.STL
- link right_shoulder_pitch: geometry visual mesh filename=new_meshes/right_shoulder_pitch.STL
- link right_shoulder_roll: geometry collision sphere radius=0.05; visual mesh filename=new_meshes/right_shoulder_roll.STL
- link right_shoulder_yaw: geometry collision cylinder length=0.14 radius=0.03; visual mesh filename=new_meshes/right_shoulder_yaw.STL
- link torso: geometry collision box size=0.14 0.18 0.28; visual mesh filename=new_meshes/torso.STL
- link waist_yaw: geometry visual mesh filename=new_meshes/waist_yaw.STL
